Commit message: lowercase update

File: URDF/FOC_URDF/urdf/FOC_URDF.urdf (robot description, URDF)
Before this commit: robot FOC_URDF, 13 links, 12 joints
Links:
- link base_link: geometry collision mesh filename=package://foc_urdf/meshes/base_link.STL; visual mesh filename=package://foc_urdf/meshes/base_link.STL
- link leg12_left: geometry collision mesh filename=package://foc_urdf/meshes/leg12_left.STL; visual mesh filename=package://foc_urdf/meshes/leg12_left.STL
- link leg1_left: geometry collision mesh filename=package://foc_urdf/meshes/leg1_left.STL; visual mesh filename=package://foc_urdf/meshes/leg1_left.STL
- link leg1_right: geometry collision mesh filename=package://foc_urdf/meshes/leg1_right.STL; visual mesh filename=package://foc_urdf/meshes/leg1_right.STL
- link leg23_left: geometry collision mesh filename=package://foc_urdf/meshes/leg23_left.STL; visual mesh filename=package://foc_urdf/meshes/leg23_left.STL
- link leg23_right: geometry collision mesh filename=package://foc_urdf/meshes/leg23_right.STL; visual mesh filename=package://foc_urdf/meshes/leg23_right.STL
- link leg2_right: geometry collision mesh filename=package://foc_urdf/meshes/leg2_right.STL; visual mesh filename=package://foc_urdf/meshes/leg2_right.STL
- link leg43_left: geometry collision mesh filename=package://foc_urdf/meshes/leg43_left.STL; visual mesh filename=package://foc_urdf/meshes/leg43_left.STL
- link leg43_right: geometry collision mesh filename=package://foc_urdf/meshes/leg43_right.STL; visual mesh filename=package://foc_urdf/meshes/leg43_right.STL
- link leg4_left: geometry collision mesh filename=package://foc_urdf/meshes/leg4_left.STL; visual mesh filename=package://foc_urdf/meshes/leg4_left.STL
- link leg4_right: geometry collision mesh filename=package://foc_urdf/meshes/leg4_right.STL; visual mesh filename=package://foc_urdf/meshes/leg4_right.STL
- link tire_left: geometry collision mesh filename=package://foc_urdf/meshes/tire_left.STL; visual mesh filename=package://foc_urdf/meshes/tire_left.STL
- link tire_right: geometry collision mesh filename=package://foc_urdf/meshes/tire_right.STL; visual mesh filename=package://foc_urdf/meshes/tire_right.STL
Joints:
- joint leg04_right: origin xyz=0.029996 -0.0665 0.03 rpy=-1.5708 0 0 -> xyz=0.0299960292290539 -0.0664999999999999 0.0300000000000001 rpy=-1.5707963267949 0 0
- joint leg12_right: origin xyz=-0.049467 -0.0072786 -0.006 rpy=0 0 0 -> xyz=-0.0494673872070477 -0.00727857148813968 -0.00600000000000005 rpy=0 0 0
- joint leg23_right: origin xyz=0.077376 0.070979 0 rpy=0 0 0 -> xyz=0.0773757935946784 0.0709787754585397 0 rpy=0 0 0
- joint leg43_left: origin xyz=-0.049424 0.0075674 0.006 rpy=0 0 0 -> xyz=-0.0494240235292409 0.00756742348365974 0.00600000000000014 rpy=0 0 0
- joint leg43_right: origin xyz=0.049967 -0.0018081 -0.006 rpy=0 0 0 -> xyz=0.0499672968829129 -0.00180810459182268 -0.00600000000000014 rpy=0 0 0
- joint tire_right: origin xyz=0.077376 0.070979 -0.0095 rpy=0 0 0 -> xyz=0.0773757935946757 0.0709787754585395 -0.00949999999999949 rpy=0 0 0
