Commit message: update

File: urdf_lowercase/foc_urdf/urdf/foc_urdf.urdf (robot description, URDF)
Before this commit: robot foc_urdf, 13 links, 12 joints
Links:
- removed link leg1_left
- removed link leg2_right
- removed link leg4_left
- removed link leg4_right
- added link leg01_left, mass 0.0077756412577186; collision mesh filename=package://foc_urdf/meshes/leg01_left.STL; visual mesh filename=package://foc_urdf/meshes/leg01_left.STL
- added link leg04_left, mass 0.0104336042175876; collision mesh filename=package://foc_urdf/meshes/leg04_left.STL; visual mesh filename=package://foc_urdf/meshes/leg04_left.STL
- added link leg04_right, mass 0.0104336042175876; collision mesh filename=package://foc_urdf/meshes/leg04_right.STL; visual mesh filename=package://foc_urdf/meshes/leg04_right.STL
- added link leg12_right, mass 0.0122831195429796; collision mesh filename=package://foc_urdf/meshes/leg12_right.STL; visual mesh filename=package://foc_urdf/meshes/leg12_right.STL
- link base_link: mass 0.310805006221372 -> 0.31081
Joints:
- removed joint leg01_left
- removed joint leg01_right
- removed joint leg04_right
- removed joint leg12_left
- removed joint leg12_right
- removed joint leg23_left
- removed joint leg23_right
- removed joint leg40_left
- removed joint leg43_left
- removed joint leg43_right
- removed joint tire_left
- removed joint tire_right
- added joint joint01_left: type revolute, parent base_link, child leg01_left, origin xyz=0.029996029229054 0.0665000000000001 0.0299999999999997 rpy=-1.5707963267949 0 0, axis 0 0 -1, limit lower=0 upper=0 effort=0 velocity=0
- added joint joint01_right: type revolute, parent base_link, child leg1_right, origin xyz=-0.0300039707709461 -0.0664999999999999 0.0300000000000001 rpy=-1.5707963267949 0 0, axis 0 0 1, limit lower=0 upper=0 effort=0 velocity=0
- added joint joint04_left: type revolute, parent base_link, child leg04_left, origin xyz=-0.0300039707709461 0.0665000000000001 0.0299999999999997 rpy=-1.5707963267949 0 0, axis 0 0 -1, limit lower=0 upper=0 effort=0 velocity=0
- added joint joint04_right: type revolute, parent base_link, child leg04_right, origin xyz=0.0299960292290539 -0.0664999999999999 0.0300000000000001 rpy=-1.5707963267949 0 0, axis 0 0 1, limit lower=0 upper=0 effort=0 velocity=0
- added joint joint12_left: type revolute, parent leg01_left, child leg12_left, origin xyz=0.0469765915200995 0.0171230794296379 0.00600000000000017 rpy=0 0 0, axis 0 0 -1, limit lower=0 upper=0 effort=0 velocity=0
- added joint joint12_right: type revolute, parent leg1_right, child leg12_right, origin xyz=-0.0494673872070477 -0.00727857148813968 -0.00600000000000005 rpy=0 0 0, axis 0 0 -1, limit lower=0 upper=0 effort=0 velocity=0
- added joint joint23_left: type revolute, parent leg12_left, child leg23_left, origin xyz=-0.083282000427136 0.0639461367469102 0 rpy=0 0 0, axis 0 0 -1, limit lower=0 upper=0 effort=0 velocity=0
- added joint joint23_right: type revolute, parent leg12_right, child leg23_right, origin xyz=0.0773757935946784 0.0709787754585397 0 rpy=0 0 0, axis 0 0 1, limit lower=0 upper=0 effort=0 velocity=0
- added joint joint43_left: type revolute, parent leg04_left, child leg43_left, origin xyz=-0.0496471723579536 0.0059294415301617 0.00600000000000026 rpy=0 0 0, axis 0 0 -1, limit lower=0 upper=0 effort=0 velocity=0
- added joint joint43_right: type revolute, parent leg04_right, child leg43_right, origin xyz=0.0499672968829129 -0.00180810459182268 -0.00600000000000014 rpy=0 0 0, axis 0 0 1, limit lower=0 upper=0 effort=0 velocity=0
- added joint joint_tire_left: type revolute, parent leg12_left, child tire_left, origin xyz=-0.0832820004271731 0.0639461367469053 0.00950000000000407 rpy=0 0 0, axis 0 0 -1, limit lower=0 upper=0 effort=0 velocity=0
- added joint joint_tire_right: type revolute, parent leg12_right, child tire_right, origin xyz=0.0773757935946757 0.0709787754585395 -0.00949999999999949 rpy=0 0 0, axis 0 0 1, limit lower=0 upper=0 effort=0 velocity=0

Commit message: fix-float

File: urdf_lowercase/foc_urdf/urdf/foc_urdf.urdf (robot description, URDF)
Before this commit: robot foc_urdf, 13 links, 12 joints
Links:
- link leg01_left: mass 0.0077756412577186 -> 0.00777564125771859
- link leg04_right: mass 0.0104336042175876 -> 0
- link leg1_right: mass 0.0077756412577186 -> 0.00777564125771859
Joints:
- joint joint01_left: origin xyz=0.029996029229054 0.0665000000000001 0.0299999999999997 rpy=-1.5707963267949 0 0 -> xyz=0.0299960292290539 0.0665000000000001 0.0299999999999997 rpy=-1.5707963267949 0 0
- joint joint01_right: origin xyz=-0.0300039707709461 -0.0664999999999999 0.0300000000000001 rpy=-1.5707963267949 0 0 -> xyz=-0.030004 -0.0665 0.03 rpy=-1.5708 0 0
- joint joint04_left: origin xyz=-0.0300039707709461 0.0665000000000001 0.0299999999999997 rpy=-1.5707963267949 0 0 -> xyz=-0.030004 0.0665 0.03 rpy=-1.5708 0 0
- joint joint04_right: origin xyz=0.0299960292290539 -0.0664999999999999 0.0300000000000001 rpy=-1.5707963267949 0 0 -> xyz=0.029996029229054 -0.0664999999999999 0.0300000000000001 rpy=-1.5707963267949 0 0
- joint joint12_left: origin xyz=0.0469765915200995 0.0171230794296379 0.00600000000000017 rpy=0 0 0 -> xyz=0.0480642169074416 0.0137779190400616 0.00600000000000019 rpy=0 0 0
- joint joint12_right: origin xyz=-0.0494673872070477 -0.00727857148813968 -0.00600000000000005 rpy=0 0 0 -> xyz=-0.0493724555181215 -0.00789687508525072 -0.00600000000000008 rpy=0 0 0
- joint joint23_left: origin xyz=-0.083282000427136 0.0639461367469102 0 rpy=0 0 0 -> xyz=-0.0824127197256137 0.0650626131309483 0 rpy=0 0 0
- joint joint23_right: origin xyz=0.0773757935946784 0.0709787754585397 0 rpy=0 0 0 -> xyz=0.0708243810933835 0.0775171403157984 0 rpy=0 0 0
- joint joint43_left: origin xyz=-0.0496471723579536 0.0059294415301617 0.00600000000000026 rpy=0 0 0 -> xyz=-0.0496751074323783 0.00569066793808726 0.00600000000000021 rpy=0 0 0
- joint joint43_right: origin xyz=0.0499672968829129 -0.00180810459182268 -0.00600000000000014 rpy=0 0 0 -> xyz=0.0487216928434121 0.0112337280754352 -0.00600000000000014 rpy=0 0 0
- joint joint_tire_left: origin xyz=-0.0832820004271731 0.0639461367469053 0.00950000000000407 rpy=0 0 0 -> xyz=-0.082412719725648 0.0650626131309466 0.00949999999999991 rpy=0 0 0
- joint joint_tire_right: origin xyz=0.0773757935946757 0.0709787754585395 -0.00949999999999949 rpy=0 0 0 -> xyz=0.0708243810933964 0.0775171403158044 -0.00949999999999991 rpy=0 0 0
