Commit message: update URDF joint

File: urdf_lowercase/foc_urdf_transmission/urdf/foc_urdf.urdf (robot description, URDF)
Before this commit: robot foc_urdf, 13 links, 12 joints
Links:
- removed link leg43_left
- removed link leg43_right
- link leg04_right: mass 0 -> 0.01
Joints:
- removed joint joint43_left
- removed joint joint43_right
- joint joint01_left: limit lower=0 upper=0 effort=0 velocity=0 -> lower=-1.57 upper=1.57 effort=0 velocity=0
- joint joint01_right: limit lower=0 upper=0 effort=0 velocity=0 -> lower=-1.57 upper=1.57 effort=0 velocity=0
- joint joint04_left: limit lower=0 upper=0 effort=0 velocity=0 -> lower=-1.57 upper=1.57 effort=0 velocity=0
- joint joint04_right: limit lower=0 upper=0 effort=0 velocity=0 -> lower=-1.57 upper=1.57 effort=0 velocity=0
- joint joint12_left: limit lower=0 upper=0 effort=0 velocity=0 -> lower=-1.57 upper=1.57 effort=0 velocity=0
- joint joint12_right: limit lower=0 upper=0 effort=0 velocity=0 -> lower=-1.57 upper=1.57 effort=0 velocity=0
- joint joint23_left: limit lower=0 upper=0 effort=0 velocity=0 -> lower=-1.57 upper=1.57 effort=0 velocity=0
- joint joint23_right: limit lower=0 upper=0 effort=0 velocity=0 -> lower=-1.57 upper=1.57 effort=0 velocity=0
- joint joint_tire_left: limit lower=0 upper=0 effort=0 velocity=0 -> lower=-1.57 upper=1.57 effort=0 velocity=0
- joint joint_tire_right: limit lower=0 upper=0 effort=0 velocity=0 -> lower=-1.57 upper=1.57 effort=0 velocity=0
