Commit message: urdf update

File: urdf/foc_urdf_transmission/urdf/foc_urdf.urdf (robot description, URDF)
Before this commit: robot foc_urdf, 11 links, 10 joints
Joints:
- joint joint01_left: limit lower=-1.57 upper=1.57 effort=0 velocity=0 -> lower=-1.396 upper=1.396 effort=20 velocity=30
- joint joint01_right: limit lower=-1.57 upper=1.57 effort=0 velocity=0 -> lower=-1.745 upper=1.745 effort=20 velocity=30
- joint joint04_left: limit lower=-1.57 upper=1.57 effort=0 velocity=0 -> lower=-1.57 upper=1.57 effort=20 velocity=30
- joint joint04_right: limit lower=-1.57 upper=1.57 effort=0 velocity=0 -> lower=-1.396 upper=1.396 effort=20 velocity=30
- joint joint12_left: limit lower=-1.57 upper=1.57 effort=0 velocity=0 -> lower=-1.57 upper=1.57 effort=20 velocity=30
- joint joint12_right: limit lower=-1.57 upper=1.57 effort=0 velocity=0 -> lower=-1.57 upper=1.57 effort=20 velocity=30
- joint joint23_left: limit lower=-1.57 upper=1.57 effort=0 velocity=0 -> lower=-1.57 upper=1.57 effort=20 velocity=30
- joint joint23_right: limit lower=-1.57 upper=1.57 effort=0 velocity=0 -> lower=-1.57 upper=1.57 effort=20 velocity=30
- joint joint_tire_left: limit lower=-1.57 upper=1.57 effort=0 velocity=0 -> lower=-1.57 upper=1.57 effort=20 velocity=30
