Commit message: try fixing LQR

File: src/urdf/foc_urdf_transmission/urdf/foc_urdf.urdf (robot description, URDF)
Before this commit: robot foc_urdf, 11 links, 10 joints
Links:
- link base_link: mass 0.31081 -> 0.58492

Commit message: small urdf fix

File: src/urdf/foc_urdf_transmission/urdf/foc_urdf.urdf (robot description, URDF)
Before this commit: robot foc_urdf, 11 links, 10 joints
Links:
- link base_link: mass 0.58492 -> 0.31081
Joints:
- joint joint_tire_right: limit lower=-1.57 upper=1.57 effort=0 velocity=0 -> lower=-1.57 upper=1.57 effort=20 velocity=30

Commit message: tuned pid

File: src/urdf/foc_urdf_transmission/urdf/foc_urdf.urdf (robot description, URDF)
Before this commit: robot foc_urdf, 11 links, 10 joints
Joints:
- joint joint_tire_right: limit lower=-1.57 upper=1.57 effort=20 velocity=30 -> lower=-1.57 upper=1.57 effort=0 velocity=0

File: src/urdf/foc_urdf_transmission/urdf/foc_urdf_old.urdf (robot description, URDF)
Before this commit: robot foc_urdf, 11 links, 10 joints
Links:
- removed link leg01_right
- removed link leg43_left
- removed link leg43_right
- added link leg1_right, mass 0.00777564125771859; collision mesh filename=package://foc_urdf/meshes/leg1_right.STL; visual mesh filename=package://foc_urdf/meshes/leg1_right.STL
- added link leg23_left, mass 0.0111561368021954; collision mesh filename=package://foc_urdf/meshes/leg23_left.STL; visual mesh filename=package://foc_urdf/meshes/leg23_left.STL
- added link leg23_right, mass 0.0111561368021954; collision mesh filename=package://foc_urdf/meshes/leg23_right.STL; visual mesh filename=package://foc_urdf/meshes/leg23_right.STL
- link leg01_left: mass 0.0077756 -> 0.00777564125771859
- link leg04_left: mass 0.010434 -> 0.0104336042175876
- link leg04_right: mass 0.010434 -> 0.01
- link leg12_left: mass 0.012283 -> 0.0122831195429796
- link leg12_right: mass 0.012283 -> 0.0122831195429796
- link tire_left: mass 0.032805 -> 0.0328045076876881
- link tire_right: mass 0.032805 -> 0.0328045076876881
Joints:
- removed joint joint43_left
- removed joint joint43_right
- added joint joint23_left: type revolute, parent leg12_left, child leg23_left, origin xyz=-0.0824127197256137 0.0650626131309483 0 rpy=0 0 0, axis 0 0 -1, limit lower=-1.57 upper=1.57 effort=20 velocity=30
- added joint joint23_right: type revolute, parent leg12_right, child leg23_right, origin xyz=0.0708243810933835 0.0775171403157984 0 rpy=0 0 0, axis 0 0 1, limit lower=-1.57 upper=1.57 effort=20 velocity=30
- joint joint01_left: limit lower=-1.919 upper=1.221 effort=0 velocity=0 -> lower=-1.396 upper=1.396 effort=20 velocity=30; origin xyz=0.0299960292290543 0.0665 0.0299999999999996 rpy=-1.5707963267949 0 0 -> xyz=0.0299960292290539 0.0665000000000001 0.0299999999999997 rpy=-1.5707963267949 0 0
- joint joint01_right: child leg01_right -> leg1_right; limit lower=-1.919 upper=1.221 effort=0 velocity=0 -> lower=-1.745 upper=1.745 effort=20 velocity=30; origin xyz=-0.0300039707709457 -0.0665 0.0299999999999996 rpy=-1.5707963267949 0 0 -> xyz=-0.030004 -0.0665 0.03 rpy=-1.5708 0 0
- joint joint04_left: limit lower=0 upper=0 effort=0 velocity=0 -> lower=-1.57 upper=1.57 effort=20 velocity=30; origin xyz=-0.0300039707709457 0.0665 0.0299999999999996 rpy=-1.5707963267949 0 0 -> xyz=-0.030004 0.0665 0.03 rpy=-1.5708 0 0
- joint joint04_right: limit lower=0 upper=0 effort=0 velocity=0 -> lower=-1.396 upper=1.396 effort=20 velocity=30; origin xyz=0.029996 -0.0665 0.03 rpy=-1.5708 0 0 -> xyz=0.029996029229054 -0.0664999999999999 0.0300000000000001 rpy=-1.5707963267949 0 0
- joint joint12_left: axis 0 0 1 -> 0 0 -1; limit lower=0 upper=0 effort=0 velocity=0 -> lower=-1.57 upper=1.57 effort=20 velocity=30; origin xyz=0.0488096092049292 0.0108453699458375 0.005 rpy=0 0 0 -> xyz=0.0480642169074416 0.0137779190400616 0.00600000000000019 rpy=0 0 0
- joint joint12_right: limit lower=0 upper=0 effort=0 velocity=0 -> lower=-1.57 upper=1.57 effort=20 velocity=30; origin xyz=-0.0492108308095336 0.00884839708848127 -0.00700000000000012 rpy=0 0 0 -> xyz=-0.0493724555181215 -0.00789687508525072 -0.00600000000000008 rpy=0 0 0; parent leg01_right -> leg1_right
- joint joint_tire_left: axis 0 0 1 -> 0 0 -1; limit lower=0 upper=0 effort=0 velocity=0 -> lower=-1.57 upper=1.57 effort=20 velocity=30; origin xyz=-0.0796741733500656 0.0683887863686989 0.0105000000000001 rpy=0 0 0 -> xyz=-0.082412719725648 0.0650626131309466 0.00949999999999991 rpy=0 0 0
- joint joint_tire_right: axis 0 0 -1 -> 0 0 1; limit lower=0 upper=0 effort=0 velocity=0 -> lower=-1.57 upper=1.57 effort=20 velocity=30; origin xyz=0.07818 0.070092 -0.0085 rpy=0 0 0 -> xyz=0.0708243810933964 0.0775171403158044 -0.00949999999999991 rpy=0 0 0
